Commit message: Update pses_robot_simple.urdf
Updated due to compability issues with ROS Melodic

File: data/urdf_model/pses_robot_simple.urdf (robot description, URDF)
Before this commit: robot pses_robot_simple, 14 links, 13 joints
Links:
- link base_footprint: geometry visual box size=0.40 0.20 0
- link base_laser: geometry visual box size=0.066 0.24 0.066
- link base_link: geometry visual box size=0.40 0.20 0.18
- link front_left_wheel: geometry visual cylinder length=0.045 radius=0.05
- link front_right_wheel: geometry visual cylinder length=0.045 radius=0.05
- link front_sensor: geometry visual box size=0.05 0.05 0.05
- link left_sensor: geometry visual box size=0.05 0.05 0.05
- link rear_left_wheel: geometry visual cylinder length=0.045 radius=0.05
- link rear_right_wheel: geometry visual cylinder length=0.045 radius=0.05
- link right_sensor: geometry visual box size=0.05 0.05 0.05
- link steering_servo: geometry visual box size=0.04 0.02 0.01
Joints:
- joint base_laser_joint: origin xyz=.18 0 .1 -> xyz=0.18 0 0.1
- joint base_link_joint: origin xyz=0 0 .1 -> xyz=0 0 0.1
- joint front_left_steering_joint: origin xyz=.14 .1 -.05 -> xyz=0.14 0.1 -0.05
- joint front_right_steering_joint: origin xyz=.14 -0.1 -.05 -> xyz=0.14 -0.1 -.05
- joint front_sensor_joint: origin xyz=.175 0 -.06 -> xyz=0.175 0 -0.06
- joint left_sensor_joint: origin xyz=0 .1 -.06 rpy=0 0 1.57 -> xyz=0 0.1 -0.06 rpy=0 0 1.57
- joint rear_left_wheel_joint: origin xyz=-.14 0.1 -.05 -> xyz=-0.14 0.1 -0.05
- joint rear_right_wheel_joint: origin xyz=-.14 -.10 -.05 -> xyz=-0.14 -0.10 -0.05
- joint right_sensor_joint: origin xyz=0 -.1 -.06 rpy=0 0 -1.57 -> xyz=0 -0.1 -0.06 rpy=0 0 -1.57
- joint steering_servo_joint: origin xyz=.08 0 -.04 -> xyz=0.08 0 -0.04

Commit message: Update pses_robot_simple.urdf

File: data/urdf_model/pses_robot_simple.urdf (robot description, URDF)
Before this commit: robot pses_robot_simple, 14 links, 13 joints
Joints:
- joint front_right_steering_joint: origin xyz=0.14 -0.1 -.05 -> xyz=0.14 -0.1 -0.05
